File: TubeTester.sch (KiCad schematic (older format))
At the start: 52 parts, among them J1 AC, Q1 IRF830, Q2 IRF830, SW1 100V/250V, SW2 100V/250V, T1 230V / 2x18V, T2 15V / 230V, U1 LM350_TO220, U2 LM317M, U3 LM317, U4 LM317

Commit message: Measurement added
Parts:
- removed J1: AC, symbol Screw_Terminal_01x02
- added J?: Tube Sockets, symbol Screw_Terminal_01x06
- added J?: Data, symbol Screw_Terminal_01x04
- added J?: AC, symbol Screw_Terminal_01x02
- added R?: 0R1, symbol R
- added R? (x2): 1R, symbol R
- added R? (x7): 1M, symbol R
- added U? (x2): ADS1015IDGS, Package_SO:TSSOP-10_3x3mm_P0.5mm, symbol ADS1015IDGS
- added U?: ISO1541, Package_SO:SOIC-8_3.9x4.9mm_P1.27mm, symbol ISO1541
- D1: value B80C3200 -> DF10
- R12, R13: value 150 -> 150R
- R6, R7: value 470 -> 470R
Connections:
- net -Ug1: now also J?.3 (Pin_3), R?.2
- net GND: now also J?.2 (Pin_2), J?.6 (Pin_6), U?.1 (ADDR), U?.3 (GND), U?.3 (GND), U?.5 (GND2)
- net Ua: now also R?.1, R?.2
- net Uf: now also R?.1, R?.2
- net Ug2: now also R?.1, R?.2
- net AC2: now reaches T1.2 (AB)
- net AC2: now also J?.2 (Pin_2)
- net AC1: now reaches F1.2
- net AC1: now also J?.1 (Pin_1)
- new net: R?.1, U?.7 (AIN3) (x2)
- new net: R?.1, U?.6 (AIN2) (x2)
- new net: R?.1, U?.5 (AIN1) (x2)
- new net: R?.1, U?.4 (AIN0)
- new net +5V: U?.8 (VCC2), U?.8 (VDD), U?.8 (VDD)
- new net +5V_Iso: U?.1 (VCC1)
- new net GND_Iso: J?.4 (Pin_4), U?.4 (GND1)
- new net SCL: U?.10 (SCL), U?.10 (SCL), U?.6 (SCL2)
- new net SCL_Iso: J?.3 (Pin_3), U?.3 (SCL1)
- new net SDA: U?.1 (ADDR), U?.7 (SDA2), U?.9 (SDA), U?.9 (SDA)
- new net SDA_Iso: J?.2 (Pin_2), U?.2 (SDA1)
- new net VCC_Iso: J?.1 (Pin_1)
- new net a: J?.5 (Pin_5), R?.2, R?.2
- new net f: J?.1 (Pin_1), R?.2, R?.2
- new net g2: J?.4 (Pin_4), R?.2, R?.2
Other:
- note added: "a"
- note added: "f"
- note added: "f'"
- note added: "g1"
- note added: "g2"
- note added: "k"
- moved on the sheet: C1, C2, C3, C4, C5, C6, C7, D1, D10, D11, D2, D3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
